File: SHVC-SOUND-ESP32-KiCad/SHVC-SOUND-ESP32.kicad_sch (KiCad schematic)
At the start: 31 parts, among them J1 PJ-324M, J3 12V in (USB-PD), J4 SHVC-SOUND module, U1 ESP32 DevKit V1 (30pin), U2 74HCT541N (data write), U3 74HCT541N (control), U4 74LVC245N (data read, DIR=B->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, U6 TDA7053A, U7 M78AR05-0.5

Commit message: ESP32版基板 r0.4: ライン出力・MUTE制御・表面ロゴシルク・GND強化
- ライン出力を追加: SHVC-SOUNDの音声 → 10µF無極性 → 47kで0V基準 → 100Ω → 端子台J5(L/GND/R)。
  アンプ(TDA7053A)とステレオジャックはそのまま
- MUTE制御: GPIO15 → 74HCT541N(U3)の空きチャンネル → SHVC-SOUND 20番。10kで引き下げ、起動中は消音
- 電源線を太く(5V系0.8mm、GND・12V・3.3V・アンプ出力0.6mm、音声0.4mm)
- GNDスティッチングビアを2mm格子で追加(表裏のGNDベタをつなぎ、島を減らす)。固定穴の周りは配線禁止
- 表面シルクにロゴ(art/logo.png → make_logo_grid.ps1 で0.1mmグリッド化)・Made by SHIMA・スペック表
- フェライトビーズFB1を10Ω(R10)に置き換え、固定穴をNPTH化

Co-Authored-By: Claude Opus 5 <noreply@anthropic.com>
Parts:
- added C14, C15: 10u NP, Capacitor_THT:CP_Radial_D4.0mm_P1.50mm, symbol SHVC-ESP32:C
- added J5: LINE OUT, TerminalBlock_Phoenix:TerminalBlock_Phoenix_PT-1,5-3-3.5-H_1x03_P3.50mm_Horizontal, symbol SHVC-ESP32:TermBlock_3
- added R11, R12: 100, Resistor_THT:R_Axial_DIN0207_L6.3mm_D2.5mm_P2.54mm_Vertical, symbol SHVC-ESP32:R
- added R13, R14: 47k, Resistor_THT:R_Axial_DIN0207_L6.3mm_D2.5mm_P2.54mm_Vertical, symbol SHVC-ESP32:R
- added R15: 10k, Resistor_THT:R_Axial_DIN0207_L6.3mm_D2.5mm_P2.54mm_Vertical, symbol SHVC-ESP32:R
Connections:
- net +5V: no longer J4.20 (~{MUTE})
- net AUDIO_L: now also C14.1 (K)
- net AUDIO_R: now also C15.1 (K)
- net GND: now also J5.2 (GND), R13.2 (A), R14.2 (A), R15.2 (A); no longer U3.7 (A6)
- net MUTE_3V3: now reaches U1.28 (IO15)
- net MUTE_3V3: now also U3.7 (A6), R15.1 (K)
- net SHVC_MUTE: now reaches U3.13 (Y6)
- net SHVC_MUTE: now also J4.20 (~{MUTE})
- new net LINE_L: J5.1 (L), R11.2 (A)
- new net LINE_R: J5.3 (R), R12.2 (A)
- new net LOUT_L: C14.2 (A), R11.1 (K), R13.1 (K)
- new net LOUT_R: C15.2 (A), R12.1 (K), R14.1 (K)
- no-connect marks 21 -> 19
Other:
- note added: "Line out J5: AUDIO -> 10uF non-polar -> 47k to GND -> 100 ohm -> terminal block (L / GND / R). No amp in path."
- note added: "MUTE: GPIO15 -> U3 A6/Y6 -> SHVC pin 20. R15 10k pulls it low = muted until firmware drives GPIO15 high."
- note added: "SHVC-SOUND player - ESP32 version (74HCT541N x2 + 74LVC245N + TDA7053A + line out)"
- note removed: "SHVC-SOUND player - ESP32 version (74HCT541N x2 + 74LVC245N + TDA7053A)"
